File: project/jalpic_one/board/jalpic_one.brd (EAGLE design)
At the start: 77.8 x 66 mm, 45 parts, among them IC1 LM2940CT-5.0, IC2 LM3940IT-3.3, IC3 PIC16F18857P, IC4 PIC16F1455P, Q1 20 MHz, Q2 12 MHz, X1 PN61729-S

Commit message: Fixed issue #227
Now also works with line endings as carriage return and line feed. Python script also updated. Next to that changed one capacitor in the schematic diagram to a typical value.
Parts:
- C10: value 220nF -> 470nF
Changed lines of the file:
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@@
 <attribute name="VALUE" x="52.959" y="14.732" size="1.27" layer="27" ratio="10" rot="R180"/>
 </element>
-<element name="C10" library="rcl" library_urn="urn:adsk.eagle:library:334" package="C050-024X044" package3d_urn="urn:adsk.eagle:package:23643/1" value="220nF" x="43.18" y="46.355" smashed="yes">
+<element name="C10" library="rcl" library_urn="urn:adsk.eagle:library:334" package="C050-024X044" package3d_urn="urn:adsk.eagle:package:23643/1" value="470nF" x="43.18" y="46.355" smashed="yes">
 <attribute name="NAME" x="41.021" y="47.752" size="1.27" layer="25" ratio="10"/>
 <attribute name="SPICEPREFIX" value="C" x="82.55" y="-4.445" size="1.778" layer="27" display="off"/>
