File: project/jalpic_one/board/jalpic_one.sch (EAGLE design)
At the start: 45 parts, among them IC1 LM2940CT-5.0, IC2 LM3940IT-3.3, IC3 PIC16F18857P, IC4 PIC16F1455P, Q1 20 MHz, Q2 12 MHz, X1 PN61729-S

Commit message: Fixed issue #227
Now also works with line endings as carriage return and line feed. Python script also updated. Next to that changed one capacitor in the schematic diagram to a typical value.
Parts:
- C10: value 220nF -> 470nF
Other:
- note added: "2019-04-05 Rob Jansen"
- note removed: "2019-03-19 Rob Jansen"
Changed lines of the file:
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@@
 <part name="C1" library="rcl" library_urn="urn:adsk.eagle:library:334" deviceset="C-EU" device="050-024X044" package3d_urn="urn:adsk.eagle:package:23643/1" value="22pF"/>
 <part name="C3" library="rcl" library_urn="urn:adsk.eagle:library:334" deviceset="C-EU" device="050-024X044" package3d_urn="urn:adsk.eagle:package:23643/1" value="22pF"/>
-<part name="C10" library="rcl" library_urn="urn:adsk.eagle:library:334" deviceset="C-EU" device="050-024X044" package3d_urn="urn:adsk.eagle:package:23643/1" value="220nF"/>
+<part name="C10" library="rcl" library_urn="urn:adsk.eagle:library:334" deviceset="C-EU" device="050-024X044" package3d_urn="urn:adsk.eagle:package:23643/1" value="470nF"/>
 <part name="C11" library="rcl" library_urn="urn:adsk.eagle:library:334" deviceset="C-EU" device="050-024X044" package3d_urn="urn:adsk.eagle:package:23643/1" value="22pF"/>
 <part name="C8" library="rcl" library_urn="urn:adsk.eagle:library:334" deviceset="C-EU" device="050-024X044" package3d_urn="urn:adsk.eagle:package:23643/1" value="100nF"/>
@@
 <plain>
 <text x="99.06" y="76.2" size="5.08" layer="91">JALPIC One</text>
-<text x="99.06" y="71.12" size="1.778" layer="91">2019-03-19
+<text x="99.06" y="71.12" size="1.778" layer="91">2019-04-05
 Rob Jansen</text>
 <text x="132.08" y="-40.64" size="1.778" layer="91">Power</text>
